Commit message: Updated Xacro model

File: simple_robotic_model/urdf/simple_model_backup.urdf.xacro (robot description, xacro)
@@ -60,5 +60,5 @@
 		<link name="second_link">
 			<visual>
-				<origin xyz="0 0 ${link_height/2}" rpy="0 0 0"/>
+				<origin xyz="0 0 0.14" rpy="0 0 0"/>
 				<geometry>
 					<box size="${link_len} ${link_width} ${link_height}"/>
@@ -66,5 +66,5 @@
 			</visual>
 			<collision>
-				<origin xyz="0 0 ${link_height/2}" rpy="0 0 0"/>
+				<origin xyz="0 0 0" rpy="0 0 0"/>
 				<geometry>
 					<box size="${link_len} ${link_width} ${link_height}"/>
@@ -78,52 +78,52 @@
 		<link name="third_link">
 			<visual>
-				<origin xyz="${link_height/2} 0 0" rpy="0 0 0"/>
+				<origin xyz="0 0.20 0" rpy="${-M_PI_HALVES} 0 0"/>
 				<geometry>
-					<box size="${link_height} ${link_width} ${link_len}"/>
+					<box size="${link_len} ${link_width} ${link_height}"/>
 				</geometry>
 			</visual>
 			<collision>
-				<origin xyz="${link_height/2} 0 0" rpy="0 0 0"/>
+				<origin xyz="0 0 0" rpy="0 0 0"/>
 				<geometry>
-					<box size="${link_height} ${link_width} ${link_len}"/>
+					<box size="${link_len} ${link_width} ${link_height}"/>
 				</geometry>
 			</collision>
-		<xacro:inertial_matrix mass="1"/>
+			<xacro:inertial_matrix mass="1"/>
 		</link>
 		<gazebo reference="third_link">
-			<material>Gazebo/Blue</material>
+			<material>Gazebo/Black</material>
 		</gazebo>
-		<link	name="fourth_link">
+		<link name="fourth_link">
 			<visual>
-				<origin xyz="${link_height/2} 0 0" rpy="0 0 0"/>
+				<origin xyz="0 0 0.14" rpy="0 0 0"/>
 				<geometry>
-					<box size="${link_height} ${link_width} ${link_len}"/>
+					<box size="${link_len} ${link_width} ${link_height}"/>
 				</geometry>
 			</visual>
 			<collision>
-				<origin xyz="${link_height/2} 0 0" rpy="0 0 0"/>
+				<origin xyz="0 0 0" rpy="0 0 0"/>
 				<geometry>
-					<box size="${link_height} ${link_width} ${link_len}"/>
+					<box size="${link_len} ${link_width} ${link_height}"/>
 				</geometry>
 			</collision>
-		<xacro:inertial_matrix mass="1"/>
+			<xacro:inertial_matrix mass="1"/>
 		</link>
 		<gazebo reference="fourth_link">
-			<material>Gazebo/Pink</material>
+			<material>Gazebo/White</material>
 		</gazebo>
 		<link name="fifth_link">
 			<visual>
-				<origin xyz="${link_height/2} 0 0" rpy="0 0 0"/>
+				<origin xyz="0 0 0.14" rpy="0 0 0"/>
 				<geometry>
-					<box size="${link_height} ${link_width} ${link_len}"/>
+					<box size="${link_len} ${link_width} ${link_height}"/>
 				</geometry>
 			</visual>
 			<collision>
-				<origin xyz="${link_height/2} 0 0" rpy="0 0 0"/>
+				<origin xyz="0 0 0" rpy="0 0 0"/>
 				<geometry>
-					<box size="${link_height} ${link_width} ${link_len}"/>
+					<box size="${link_len} ${link_width} ${link_height}"/>
 				</geometry>
 			</collision>
-		<xacro:inertial_matrix mass="1"/>
+			<xacro:inertial_matrix mass="1"/>
 		</link>
 		<gazebo reference="fifth_link">
@@ -132,19 +132,19 @@
 		<link name="sixth_link">
 			<visual>
-				<origin xyz="${link_height/2} 0 0" rpy="0 0 0"/>
+				<origin xyz="0 0 0.14" rpy="0 0 0"/>
 				<geometry>
-					<box size="${link_height} ${link_width} ${link_len}"/>
+					<box size="${link_len} ${link_width} ${link_height}"/>
 				</geometry>
 			</visual>
 			<collision>
-				<origin xyz="${link_height/2} 0 0" rpy="0 0 0"/>
+				<origin xyz="0 0 0" rpy="0 0 0"/>
 				<geometry>
-					<box size="${link_height} ${link_width} ${link_len}"/>
+					<box size="${link_len} ${link_width} ${link_height}"/>
 				</geometry>
 			</collision>
-		<xacro:inertial_matrix mass="1"/>
+			<xacro:inertial_matrix mass="1"/>
 		</link>
 		<gazebo reference="sixth_link">
-			<material>Gazebo/Black</material>
+			<material>Gazebo/Blue</material>
 		</gazebo>
 		<joint name="fixed" type="fixed">
@@ -153,5 +153,5 @@
 		</joint>
 		<joint name="second_joint" type="revolute">
-			<origin xyz="0 0 0.15" rpy="0 0 0"/>
+			<origin xyz="0 0 0.1" rpy="0 0 0"/>
 			<parent link="base_link"/>
 			<child link="second_link"/>
@@ -160,30 +160,30 @@
 		</joint>
 		<joint name="third_joint" type="revolute">
-			<origin xyz="0 0 0.26" rpy="0 ${-M_PI_HALVES} 0"/>
+			<origin xyz="0 0 0.26" rpy="${M_PI_HALVES} 0 0"/>
 			<parent link="second_link"/>
 			<child link="third_link"/>
-			<axis xyz="0 0 1"/>
-			<limit effort="300" velocity="1" lower="${-M_PI_HALVES}" upper="${M_PI_HALVES}"/>
+			<axis xyz="0 1 0"/>
+			<limit effort="300" velocity="1" lower="0" upper="${M_PI}"/>
 		</joint>
 		<joint name="fourth_joint" type="revolute">
-			<origin xyz="0.26 0 0" rpy="0 0 0"/>
+			<origin xyz="0 0 0.26" rpy="0 0 0"/>
 			<parent link="third_link"/>
 			<child link="fourth_link"/>
-			<axis xyz="0 0 1"/>
-			<limit effort="300" velocity="1" lower="${-M_PI_HALVES}" upper="${M_PI_HALVES}"/>
+			<axis xyz="1 0 0"/>
+			<limit effort="300" velocity="1" lower="0" upper="${M_PI}"/>
 		</joint>
 		<joint name="fifth_joint" type="revolute">
-			<origin xyz="0.26 0 0" rpy="0 0 0"/>
+			<origin xyz="0 0 0.26" rpy="0 0 0"/>
 			<parent link="fourth_link"/>
 			<child link="fifth_link"/>
-			<axis xyz="0 0 1"/>
-			<limit effort="300" velocity="1" lower="${-M_PI_HALVES}" upper="${M_PI_HALVES}"/>
+			<axis xyz="1 0 0"/>
+			<limit effort="300" velocity="1" lower="0" upper="${M_PI}"/>
 		</joint>
 		<joint name="sixth_joint" type="revolute">
-			<origin xyz="0.26 0 0" rpy="0 0 0"/>
+			<origin xyz="0 0 0.26" rpy="0 0 0"/>
 			<parent link="fifth_link"/>
 			<child link="sixth_link"/>
-			<axis xyz="0 0 1"/>
-			<limit effort="300" velocity="1" lower="${-M_PI_HALVES}" upper="${M_PI_HALVES}"/>
+			<axis xyz="1 0 0"/>
+			<limit effort="300" velocity="1" lower="0" upper="${M_PI}"/>
 		</joint>
 		<xacro:transmission_block joint_name="second_joint"/>

File: simple_robotic_model/urdf/simple_model_generated.urdf (robot description, URDF)
Before this commit: robot simple_model, 7 links, 6 joints
Links:
- removed link bottom_link
- added link world
- link fifth_link: geometry collision box size=0.2 0.1 0.1; visual box size=0.2 0.1 0.1
- link fourth_link: geometry collision box size=0.2 0.1 0.1; visual box size=0.2 0.1 0.1
- link sixth_link: geometry collision box size=0.2 0.1 0.1; visual box size=0.2 0.1 0.1
- link third_link: geometry collision box size=0.2 0.1 0.1; visual box size=0.2 0.1 0.1
Joints:
- removed joint bottom_joint
- added joint fixed: type fixed, parent world, child base_link
- joint fifth_joint: axis 1 0 0 -> 0 0 1; limit lower=-1.0 upper=1.0 effort=300 velocity=1 -> lower=-1.570795 upper=1.570795 effort=300 velocity=1; origin xyz=0 0 0.26 rpy=0 0 0 -> xyz=0.26 0 0 rpy=0 0 0
- joint fourth_joint: axis 1 0 0 -> 0 0 1; limit lower=-1.0 upper=1.0 effort=300 velocity=1 -> lower=-1.570795 upper=1.570795 effort=300 velocity=1; origin xyz=0 0 0.26 rpy=0 0 0 -> xyz=0.26 0 0 rpy=0 0 0
- joint second_joint: limit lower=-1.0 upper=1.0 effort=300 velocity=1 -> lower=0 upper=3.14159 effort=300 velocity=1; origin xyz=0 0 0.1 rpy=0 0 0 -> xyz=0 0 0.15 rpy=0 0 0
- joint sixth_joint: axis 1 0 0 -> 0 0 1; limit lower=-1.0 upper=1.0 effort=300 velocity=1 -> lower=-1.570795 upper=1.570795 effort=300 velocity=1; origin xyz=0 0 0.26 rpy=0 0 0 -> xyz=0.26 0 0 rpy=0 0 0
- joint third_joint: axis 1 0 0 -> 0 0 1; limit lower=-1.0 upper=1.0 effort=300 velocity=1 -> lower=-1.570795 upper=1.570795 effort=300 velocity=1; origin xyz=0 0 0.26 rpy=0 0 0 -> xyz=0 0 0.26 rpy=0 -1.570795 0
