Commit message: Changes to Z and generated URDF

File: simple_robotic_model/urdf/simple_model_generated.urdf (robot description, URDF)
Before this commit: robot simple_model, 12 links, 11 joints
Joints:
- joint third_joint: limit lower=-1.04719755 upper=1.04719755 effort=300 velocity=1 -> lower=-0.7853975 upper=-0.7853975 effort=300 velocity=1
