Commit message: Configured xacro model

File: simple_robotic_model/urdf/simple_model.urdf.xacro (robot description, xacro)
@@ -3,5 +3,5 @@
 	<!-- Include materials -->
 		<material name="Black">
-			<color rgba="0.0 0.0 0.0 1.0"/>
+			<color rgba="0.5 0.0 0.0 1.0"/>
 		</material>
 		<material name="Red">
@@ -147,4 +147,22 @@
 			<material>Gazebo/Black</material>
 		</gazebo>
+		<link name="sixth_link">
+			<visual>
+				<origin xyz="0 0 0.14" rpy="0 0 0"/>
+				<geometry>
+					<box size="${link_len} ${link_width} ${link_height}"/>
+				</geometry>
+			</visual>
+			<collision>
+				<origin xyz="0 0 0" rpy="0 0 0"/>
+				<geometry>
+					<box size="${link_len} ${link_width} ${link_height}"/>
+				</geometry>
+			</collision>
+			<xacro:inertial_matrix mass="1"/>
+		</link>
+		<gazebo reference="sixth_link">
+			<material>Gazebo/Blue</material>
+		</gazebo>
 		<joint name="bottom_joint" type="fixed">
 			<origin xyz="0 0 -0.04" rpy="0 0 0"/>
@@ -177,4 +195,11 @@
 			<parent link="fourth_link"/>
 			<child link="fifth_link"/>
+			<axis xyz="1 0 0"/>
+			<limit effort="300" velocity="1" lower="-1.0" upper="1.0"/>
+		</joint>
+		<joint name="sixth_joint" type="revolute">
+			<origin xyz="0 0 0.26" rpy="0 0 0"/>
+			<parent link="fifth_link"/>
+			<child link="sixth_link"/>
 			<axis xyz="1 0 0"/>
 			<limit effort="300" velocity="1" lower="-1.0" upper="1.0"/>

File: simple_robotic_model/urdf/simple_model_generated.urdf (robot description, URDF)
Before this commit: robot simple_model, 6 links, 5 joints
Links:
- added link sixth_link, mass 1; collision box size=0.1 0.1 0.2; visual box size=0.1 0.1 0.2
Joints:
- added joint sixth_joint: type revolute, parent fifth_link, child sixth_link, origin xyz=0 0 0.26 rpy=0 0 0, axis 1 0 0, limit lower=-1.0 upper=1.0 effort=300 velocity=1
- joint third_joint: axis 0 1 0 -> 1 0 0

Commit message: Inverse kinematics with Matlab

File: simple_robotic_model/urdf/simple_model.urdf.xacro (robot description, xacro)
@@ -148,4 +148,22 @@
 			<material>Gazebo/Black</material>
 		</gazebo>
+		<link name="end_effector">
+			<visual>
+				<origin xyz="0 0 0" rpy="0 0 0"/>
+				<geometry>
+					<box size="0.05 0.05 0.05"/>
+				</geometry>
+			</visual>
+			<collision>
+				<origin xyz="0 0 0" rpy="0 0 0"/>
+				<geometry>
+					<box size="0.05 0.05 0.05"/>
+				</geometry>
+			</collision>
+			<xacro:inertial_matrix mass="1"/>
+			</link>
+			<gazebo reference="end_effector">
+				<material>Gazebo/Blue</material>
+			</gazebo>
 		<joint name="fixed" type="fixed">
 			<parent link="world"/>
@@ -186,4 +204,9 @@
 			<axis xyz="0 0 1"/>
 			<limit effort="300" velocity="1" lower="${-M_PI_HALVES}" upper="${M_PI_HALVES}"/>
+		</joint>
+		<joint name="ee_joint" type="fixed">
+			<origin xyz="0.26 0 0" rpy="0 0 0"/>
+			<parent link="sixth_link"/>
+			<child link="end_effector"/>
 		</joint>
 		<xacro:transmission_block joint_name="second_joint"/>

File: simple_robotic_model/urdf/simple_model_generated.urdf (robot description, URDF)
Before this commit: robot simple_model, 7 links, 6 joints
Links:
- added link end_effector, mass 1; collision box size=0.05 0.05 0.05; visual box size=0.05 0.05 0.05
Joints:
- added joint ee_joint: type fixed, parent sixth_link, child end_effector, origin xyz=0.26 0 0 rpy=0 0 0

Commit message: Redesign of URDF with real measurements

File: simple_robotic_model/urdf/simple_model.urdf.xacro (robot description, xacro)
@@ -16,7 +16,11 @@
 		<xacro:property name="M_PI_HALVES" value="${M_PI / 2}"/>
 		<!-- Second link properties -->
-		<xacro:property name="link_len" value="0.1"/>
-		<xacro:property name="link_width" value="0.1"/>
-		<xacro:property name="link_height" value="0.2"/>
+		<xacro:property name="link_len" value="0.035"/>
+		<xacro:property name="link_width" value="0.03"/>
+		<xacro:property name="second_link_height" value="0.036"/>
+		<xacro:property name="third_link_height" value="0.029"/>
+		<xacro:property name="fourth_link_height" value="0.069"/>
+		<xacro:property name="fifth_link_height" value="0.027"/>
+		<xacro:property name="ee_link_height" value="0.02"/>
 		<xacro:macro name="inertial_matrix" params="mass">
 			<inertial>
@@ -41,14 +45,14 @@
 		<link name="base_link">
 			<visual>
-				<origin xyz="0 0 0.05" rpy="0 0 0"/>
-				<geometry>
-					<box size="0.1 0.1 0.1"/>
+				<origin xyz="0 0 0.005" rpy="0 0 0"/>
+				<geometry>
+					<box size="0.1 0.1 0.01"/>
 				</geometry>
 				<material name="White"/>
 			</visual>
 			<collision>
-				<origin xyz="0 0 0.05" rpy="0 0 0"/>
-				<geometry>
-					<box size="0.1 0.1 0.1"/>
+				<origin xyz="0 0 0.005" rpy="0 0 0"/>
+				<geometry>
+					<box size="0.1 0.1 0.01"/>
 				</geometry>
 			</collision>
@@ -56,17 +60,34 @@
 		</link>
 		<gazebo reference="base_link">
-			<material>Gazebo/Yellow</material>
+			<material>Gazebo/Black</material>
+		</gazebo>
+		<link name="second_joint_placeholder">
+			<visual>
+				<origin xyz="0 0 0.0095" rpy="0 0 0"/>
+				<geometry>
+					<cylinder length="0.021" radius="0.025"/>
+				</geometry>
+			</visual>
+			<collision>
+				<origin xyz="0 0 0.0095" rpy="0 0 0"/>
+				<geometry>
+					<cylinder length="0.021" radius="0.025"/>
+				</geometry>
+			</collision>
+		</link>
+		<gazebo reference="second_joint_placeholder">
+			<material>Gazebo/Orange</material>
 		</gazebo>
 		<link name="second_link">
 			<visual>
-				<origin xyz="0 0 ${link_height/2}" rpy="0 0 0"/>
-				<geometry>
-					<box size="${link_len} ${link_width} ${link_height}"/>
-				</geometry>
-			</visual>
-			<collision>
-				<origin xyz="0 0 ${link_height/2}" rpy="0 0 0"/>
-				<geometry>
-					<box size="${link_len} ${link_width} ${link_height}"/>
+				<origin xyz="0 0 0.039" rpy="0 0 0"/>
+				<geometry>
+					<box size="${link_len} ${link_width} ${second_link_height}"/>
+				</geometry>
+			</visual>
+			<collision>
+				<origin xyz="0 0 0.039" rpy="0 0 0"/>
+				<geometry>
+					<box size="${link_len} ${link_width} ${second_link_height}"/>
 				</geometry>
 			</collision>
@@ -74,17 +95,34 @@
 		</link>
 		<gazebo reference="second_link">
-			<material>Gazebo/Green</material>
+			<material>Gazebo/Black</material>
+		</gazebo>
+		<link name="third_joint_placeholder">
+			<visual>
+				<origin xyz="0 0 0" rpy="0 0 0"/>
+				<geometry>
+					<cylinder length="0.05" radius="0.025"/>
+				</geometry>
+			</visual>
+			<collision>
+				<origin xyz="0 0 0" rpy="1 0 0"/>
+				<geometry>
+					<cylinder length="0.05" radius="0.025"/>
+				</geometry>
+			</collision>
+		</link>
+		<gazebo reference="third_joint_placeholder">
+			<material>Gazebo/Orange</material>
 		</gazebo>
 		<link name="third_link">
 			<visual>
-				<origin xyz="${link_height/2} 0 0" rpy="0 0 0"/>
-				<geometry>
-					<box size="${link_height} ${link_width} ${link_len}"/>
-				</geometry>
-			</visual>
-			<collision>
-				<origin xyz="${link_height/2} 0 0" rpy="0 0 0"/>
-				<geometry>
-					<box size="${link_height} ${link_width} ${link_len}"/>
+				<origin xyz="0 0 0" rpy="0 0 0"/>
+				<geometry>
+					<box size="${third_link_height} ${link_width} ${link_len}"/>
+				</geometry>
+			</visual>
+			<collision>
+				<origin xyz="0 0 0" rpy="0 0 0"/>
+				<geometry>
+					<box size="${third_link_height} ${link_width} ${link_len}"/>
 				</geometry>
 			</collision>
@@ -92,59 +130,95 @@
 		</link>
 		<gazebo reference="third_link">
-			<material>Gazebo/Blue</material>
-		</gazebo>
-		<link	name="fourth_link">
-			<visual>
-				<origin xyz="${link_height/2} 0 0" rpy="0 0 0"/>
-				<geometry>
-					<box size="${link_height} ${link_width} ${link_len}"/>
-				</geometry>
-			</visual>
-			<collision>
-				<origin xyz="${link_height/2} 0 0" rpy="0 0 0"/>
-				<geometry>
-					<box size="${link_height} ${link_width} ${link_len}"/>
-				</geometry>
-			</collision>
-		<xacro:inertial_matrix mass="1"/>
+			<material>Gazebo/Black</material>
+		</gazebo>
+		<link name="fourth_joint_placeholder">
+			<visual>
+				<origin xyz="0 0 0" rpy="0 0 0"/>
+				<geometry>
+					<cylinder length="0.05" radius="0.025"/>
+				</geometry>
+			</visual>
+			<collision>
+				<origin xyz="0 0 0" rpy="0 0 0"/>
+				<geometry>
+					<cylinder length="0.05" radius="0.025"/>
+				</geometry>
+			</collision>
+			<xacro:inertial_matrix mass="1"/>
+		</link>
+		<gazebo reference="fourth_joint_placeholder">
+			<material>Gazebo/Orange</material>
+		</gazebo>
+		<link name="fourth_link">
+			<visual>
+				<origin xyz="0 0 0" rpy="0 0 0"/>
+				<geometry>
+					<box size="${fourth_link_height} ${link_width} ${link_len}"/>
+				</geometry>
+			</visual>
+			<collision>
+				<origin xyz="0 0 0" rpy="0 0 0"/>
+				<geometry>
+					<box size="${fourth_link_height} ${link_width} ${link_len}"/>
+				</geometry>
+			</collision>
+			<xacro:inertial_matrix mass="1"/>
 		</link>
 		<gazebo reference="fourth_link">
-			<material>Gazebo/Pink</material>
+			<material>Gazebo/Black</material>
+		</gazebo>
+		<link name="fifth_joint_placeholder">
+			<visual>
+				<origin xyz="0 0 0" rpy="0 0 0"/>
+				<geometry>
+					<cylinder length="0.05" radius="0.025"/>
+				</geometry>
+			</visual>
+			<collision>
+				<origin xyz="0 0 0" rpy="0 0 0"/>
+				<geometry>
+					<cylinder length="0.05" radius="0.025"/>
+				</geometry>
+			</collision>
+			<xacro:inertial_matrix mass="1"/>
+		</link>
+		<gazebo reference="fifth_joint_placeholder">
+			<material>Gazebo/Orange</material>
 		</gazebo>
 		<link name="fifth_link">
 			<visual>
-				<origin xyz="${link_height/2} 0 0" rpy="0 0 0"/>
-				<geometry>
-					<box size="${link_height} ${link_width} ${link_len}"/>
-				</geometry>
-			</visual>
-			<collision>
-				<origin xyz="${link_height/2} 0 0" rpy="0 0 0"/>
-				<geometry>
-					<box size="${link_height} ${link_width} ${link_len}"/>
-				</geometry>
-			</collision>
-		<xacro:inertial_matrix mass="1"/>
+				<origin xyz="0 0 0" rpy="0 0 0"/>
+				<geometry>
+					<box size="${fifth_link_height} ${link_width} ${link_len}"/>
+				</geometry>
+			</visual>
+			<collision>
+				<origin xyz="0 0 0" rpy="0 0 0"/>
+				<geometry>
+					<box size="${fifth_link_height} ${link_width} ${link_len}"/>
+				</geometry>
+			</collision>
+			<xacro:inertial_matrix mass="1"/>
 		</link>
 		<gazebo reference="fifth_link">
 			<material>Gazebo/Black</material>
 		</gazebo>
-		<link name="sixth_link">
-			<visual>
-				<origin xyz="${link_height/2} 0 0" rpy="0 0 0"/>
-				<geometry>
-					<box size="${link_height} ${link_width} ${link_len}"/>
-				</geometry>
-			</visual>
-			<collision>
-				<origin xyz="${link_height/2} 0 0" rpy="0 0 0"/>
-				<geometry>
-					<box size="${link_height} ${link_width} ${link_len}"/>
-				</geometry>
-			</collision>
-		<xacro:inertial_matrix mass="1"/>
-		</link>
-		<gazebo reference="sixth_link">
-			<material>Gazebo/Black</material>
+		<link name="sixth_joint_placeholder">
+			<visual>
+				<origin xyz="0 0 0" rpy="0 0 0"/>
+				<geometry>
+					<cylinder length="0.05" radius="0.02"/>
+				</geometry>
+			</visual>
+			<collision>
+				<origin xyz="0 0 0" rpy="0 0 0"/>
+				<geometry>
+					<cylinder length="0.05" radius="0.02"/>
+				</geometry>
+			</collision>
+			<xacro:inertial_matrix mass="1"/>
+		</link>
+		<gazebo reference="sixth_joint_placeholder">
+			<material>Gazebo/Orange</material>
 		</gazebo>
 		<link name="end_effector">
@@ -152,18 +226,19 @@
 				<origin xyz="0 0 0" rpy="0 0 0"/>
 				<geometry>
-					<box size="0.05 0.05 0.05"/>
-				</geometry>
-			</visual>
-			<collision>
-				<origin xyz="0 0 0" rpy="0 0 0"/>
-				<geometry>
-					<box size="0.05 0.05 0.05"/>
-				</geometry>
-			</collision>
-			<xacro:inertial_matrix mass="1"/>
-			</link>
-			<gazebo reference="end_effector">
-				<material>Gazebo/Blue</material>
-			</gazebo>
+					<box size="${ee_link_height} 0.010 0.015"/>
+				</geometry>
+			</visual>
+			<collision>
+				<origin xyz="0 0 0" rpy="0 0 0"/>
+				<geometry>
+					<box size="${ee_link_height} 0.010 0.015"/>
+				</geometry>
+			</collision>
+			<xacro:inertial_matrix mass="1"/>
+		</link>
+		<gazebo reference="end_effector">
+			<material>Gazebo/Black</material>
+		</gazebo>
+		<!-- JOINTS -->
 		<joint name="fixed" type="fixed">
 			<parent link="world"/>
@@ -171,41 +246,60 @@
 		</joint>
 		<joint name="second_joint" type="revolute">
-			<origin xyz="0 0 0.15" rpy="0 0 0"/>
+			<origin xyz="0 0 0.01" rpy="0 0 0"/>
 			<parent link="base_link"/>
+			<child link="second_joint_placeholder"/>
+			<axis xyz="0 0 1"/>
+			<limit effort="300" velocity="1" lower="0" upper="${M_PI}"/>
+		</joint>
+		<joint name="second_fixed" type="fixed">
+			<parent link="second_joint_placeholder"/>
 			<child link="second_link"/>
-			<axis xyz="0 0 1"/>
-			<limit effort="300" velocity="1" lower="0" upper="${M_PI}"/>
 		</joint>
 		<joint name="third_joint" type="revolute">
-			<origin xyz="0 0 0.26" rpy="0 ${-M_PI_HALVES} 0"/>
+			<origin xyz="0 0 0.076" rpy="0 ${-M_PI_HALVES} 0"/>
 			<parent link="second_link"/>
+			<child link="third_joint_placeholder"/>
+			<axis xyz="0 0 1"/>
+			<limit effort="300" velocity="1" lower="${-M_PI_HALVES}" upper="${M_PI_HALVES}"/>
+		</joint>
+		<joint name="third_fixed" type="fixed">
+			<origin xyz="0.034 0 0" rpy="0 0 0"/> <!-- Radius 0.03 -->
+			<parent link="third_joint_placeholder"/>
 			<child link="third_link"/>
+		</joint>
+		<joint name="fourth_joint" type="revolute">
+			<origin xyz="0.035 0 0" rpy="0 0 0"/>
+			<parent link="third_link"/>
+			<child link="fourth_joint_placeholder"/>
 			<axis xyz="0 0 1"/>
 			<limit effort="300" velocity="1" lower="${-M_PI_HALVES}" upper="${M_PI_HALVES}"/>
 		</joint>
-		<joint name="fourth_joint" type="revolute">
-			<origin xyz="0.26 0 0" rpy="0 0 0"/>
-			<parent link="third_link"/>
+		<joint name="fourth_fixed" type="fixed">
+			<origin xyz="0.054 0 0" rpy="0 0 0"/>
+			<parent link="fourth_joint_placeholder"/>
 			<child link="fourth_link"/>
+		</joint>
+		<joint name="fifth_joint" type="revolute">
+			<origin xyz="0.055 0 0" rpy="0 0 0"/>
+			<parent link="fourth_link"/>
+			<child link="fifth_joint_placeholder"/>
 			<axis xyz="0 0 1"/>
 			<limit effort="300" velocity="1" lower="${-M_PI_HALVES}" upper="${M_PI_HALVES}"/>
 		</joint>
-		<joint name="fifth_joint" type="revolute">
-			<origin xyz="0.26 0 0" rpy="0 0 0"/>
-			<parent link="fourth_link"/>
+		<joint name="fifth_fixed" type="fixed">
+			<origin xyz="0.034 0 0" rpy="0 0 0"/>
+			<parent link="fifth_joint_placeholder"/>
 			<child link="fifth_link"/>
+		</joint>
+		<joint name="sixth_joint" type="revolute">
+			<origin xyz="0.0275 0 0" rpy="0 0 0"/>
+			<parent link="fifth_link"/>
+			<child link="sixth_joint_placeholder"/>
 			<axis xyz="0 0 1"/>
 			<limit effort="300" velocity="1" lower="${-M_PI_HALVES}" upper="${M_PI_HALVES}"/>
 		</joint>
-		<joint name="sixth_joint" type="revolute">
-			<origin xyz="0.26 0 0" rpy="0 0 0"/>
-			<parent link="fifth_link"/>
-			<child link="sixth_link"/>
-			<axis xyz="0 0 1"/>
-			<limit effort="300" velocity="1" lower="${-M_PI_HALVES}" upper="${M_PI_HALVES}"/>
-		</joint>
 		<joint name="ee_joint" type="fixed">
-			<origin xyz="0.26 0 0" rpy="0 0 0"/>
-			<parent link="sixth_link"/>
+			<origin xyz="0.029 0 0" rpy="0 0 0"/>
+			<parent link="sixth_joint_placeholder"/>
 			<child link="end_effector"/>
 		</joint>
