Commit message: Redesign of URDF with real measurements

File: simple_robotic_model/urdf/simple_model_backup.urdf.xacro (robot description, xacro)
@@ -16,7 +16,11 @@
 		<xacro:property name="M_PI_HALVES" value="${M_PI / 2}"/>
 		<!-- Second link properties -->
-		<xacro:property name="link_len" value="0.1"/>
-		<xacro:property name="link_width" value="0.1"/>
-		<xacro:property name="link_height" value="0.2"/>
+		<xacro:property name="link_len" value="0.035"/>
+		<xacro:property name="link_width" value="0.03"/>
+		<xacro:property name="second_link_height" value="0.036"/>
+		<xacro:property name="third_link_height" value="0.029"/>
+		<xacro:property name="fourth_link_height" value="0.069"/>
+		<xacro:property name="fifth_link_height" value="0.027"/>
+		<xacro:property name="ee_link_height" value="0.02"/>
 		<xacro:macro name="inertial_matrix" params="mass">
 			<inertial>
@@ -41,14 +45,14 @@
 		<link name="base_link">
 			<visual>
-				<origin xyz="0 0 0.05" rpy="0 0 0"/>
-				<geometry>
-					<box size="0.1 0.1 0.1"/>
+				<origin xyz="0 0 0.005" rpy="0 0 0"/>
+				<geometry>
+					<box size="0.1 0.1 0.01"/>
 				</geometry>
 				<material name="White"/>
 			</visual>
 			<collision>
-				<origin xyz="0 0 0.05" rpy="0 0 0"/>
-				<geometry>
-					<box size="0.1 0.1 0.1"/>
+				<origin xyz="0 0 0.005" rpy="0 0 0"/>
+				<geometry>
+					<box size="0.1 0.1 0.01"/>
 				</geometry>
 			</collision>
@@ -56,17 +60,34 @@
 		</link>
 		<gazebo reference="base_link">
-			<material>Gazebo/Yellow</material>
+			<material>Gazebo/Black</material>
+		</gazebo>
+		<link name="second_joint_placeholder">
+			<visual>
+				<origin xyz="0 0 0.0095" rpy="0 0 0"/>
+				<geometry>
+					<cylinder length="0.021" radius="0.025"/>
+				</geometry>
+			</visual>
+			<collision>
+				<origin xyz="0 0 0.0095" rpy="0 0 0"/>
+				<geometry>
+					<cylinder length="0.021" radius="0.025"/>
+				</geometry>
+			</collision>
+		</link>
+		<gazebo reference="second_joint_placeholder">
+			<material>Gazebo/Orange</material>
 		</gazebo>
 		<link name="second_link">
 			<visual>
-				<origin xyz="0 0 0.14" rpy="0 0 0"/>
-				<geometry>
-					<box size="${link_len} ${link_width} ${link_height}"/>
-				</geometry>
-			</visual>
-			<collision>
-				<origin xyz="0 0 0" rpy="0 0 0"/>
-				<geometry>
-					<box size="${link_len} ${link_width} ${link_height}"/>
+				<origin xyz="0 0 0.039" rpy="0 0 0"/>
+				<geometry>
+					<box size="${link_len} ${link_width} ${second_link_height}"/>
+				</geometry>
+			</visual>
+			<collision>
+				<origin xyz="0 0 0.039" rpy="0 0 0"/>
+				<geometry>
+					<box size="${link_len} ${link_width} ${second_link_height}"/>
 				</geometry>
 			</collision>
@@ -74,35 +95,70 @@
 		</link>
 		<gazebo reference="second_link">
-			<material>Gazebo/Green</material>
+			<material>Gazebo/Black</material>
+		</gazebo>
+		<link name="third_joint_placeholder">
+			<visual>
+				<origin xyz="0 0 0" rpy="0 0 0"/>
+				<geometry>
+					<cylinder length="0.05" radius="0.025"/>
+				</geometry>
+			</visual>
+			<collision>
+				<origin xyz="0 0 0" rpy="1 0 0"/>
+				<geometry>
+					<cylinder length="0.05" radius="0.025"/>
+				</geometry>
+			</collision>
+		</link>
+		<gazebo reference="third_joint_placeholder">
+			<material>Gazebo/Orange</material>
 		</gazebo>
 		<link name="third_link">
 			<visual>
-				<origin xyz="0 0.20 0" rpy="${-M_PI_HALVES} 0 0"/>
-				<geometry>
-					<box size="${link_len} ${link_width} ${link_height}"/>
-				</geometry>
-			</visual>
-			<collision>
-				<origin xyz="0 0 0" rpy="0 0 0"/>
-				<geometry>
-					<box size="${link_len} ${link_width} ${link_height}"/>
-				</geometry>
-			</collision>
-			<xacro:inertial_matrix mass="1"/>
+				<origin xyz="0 0 0" rpy="0 0 0"/>
+				<geometry>
+					<box size="${third_link_height} ${link_width} ${link_len}"/>
+				</geometry>
+			</visual>
+			<collision>
+				<origin xyz="0 0 0" rpy="0 0 0"/>
+				<geometry>
+					<box size="${third_link_height} ${link_width} ${link_len}"/>
+				</geometry>
+			</collision>
+		<xacro:inertial_matrix mass="1"/>
 		</link>
 		<gazebo reference="third_link">
 			<material>Gazebo/Black</material>
 		</gazebo>
+		<link name="fourth_joint_placeholder">
+			<visual>
+				<origin xyz="0 0 0" rpy="0 0 0"/>
+				<geometry>
+					<cylinder length="0.05" radius="0.025"/>
+				</geometry>
+			</visual>
+			<collision>
+				<origin xyz="0 0 0" rpy="0 0 0"/>
+				<geometry>
+					<cylinder length="0.05" radius="0.025"/>
+				</geometry>
+			</collision>
+			<xacro:inertial_matrix mass="1"/>
+		</link>
+		<gazebo reference="fourth_joint_placeholder">
+			<material>Gazebo/Orange</material>
+		</gazebo>
 		<link name="fourth_link">
 			<visual>
-				<origin xyz="0 0 0.14" rpy="0 0 0"/>
-				<geometry>
-					<box size="${link_len} ${link_width} ${link_height}"/>
-				</geometry>
-			</visual>
-			<collision>
-				<origin xyz="0 0 0" rpy="0 0 0"/>
-				<geometry>
-					<box size="${link_len} ${link_width} ${link_height}"/>
+				<origin xyz="0 0 0" rpy="0 0 0"/>
+				<geometry>
+					<box size="${fourth_link_height} ${link_width} ${link_len}"/>
+				</geometry>
+			</visual>
+			<collision>
+				<origin xyz="0 0 0" rpy="0 0 0"/>
+				<geometry>
+					<box size="${fourth_link_height} ${link_width} ${link_len}"/>
 				</geometry>
 			</collision>
@@ -110,17 +166,35 @@
 		</link>
 		<gazebo reference="fourth_link">
-			<material>Gazebo/White</material>
+			<material>Gazebo/Black</material>
+		</gazebo>
+		<link name="fifth_joint_placeholder">
+			<visual>
+				<origin xyz="0 0 0" rpy="0 0 0"/>
+				<geometry>
+					<cylinder length="0.05" radius="0.025"/>
+				</geometry>
+			</visual>
+			<collision>
+				<origin xyz="0 0 0" rpy="0 0 0"/>
+				<geometry>
+					<cylinder length="0.05" radius="0.025"/>
+				</geometry>
+			</collision>
+			<xacro:inertial_matrix mass="1"/>
+		</link>
+		<gazebo reference="fifth_joint_placeholder">
+			<material>Gazebo/Orange</material>
 		</gazebo>
 		<link name="fifth_link">
 			<visual>
-				<origin xyz="0 0 0.14" rpy="0 0 0"/>
-				<geometry>
-					<box size="${link_len} ${link_width} ${link_height}"/>
-				</geometry>
-			</visual>
-			<collision>
-				<origin xyz="0 0 0" rpy="0 0 0"/>
-				<geometry>
-					<box size="${link_len} ${link_width} ${link_height}"/>
+				<origin xyz="0 0 0" rpy="0 0 0"/>
+				<geometry>
+					<box size="${fifth_link_height} ${link_width} ${link_len}"/>
+				</geometry>
+			</visual>
+			<collision>
+				<origin xyz="0 0 0" rpy="0 0 0"/>
+				<geometry>
+					<box size="${fifth_link_height} ${link_width} ${link_len}"/>
 				</geometry>
 			</collision>
@@ -130,22 +204,41 @@
 			<material>Gazebo/Black</material>
 		</gazebo>
-		<link name="sixth_link">
-			<visual>
-				<origin xyz="0 0 0.14" rpy="0 0 0"/>
-				<geometry>
-					<box size="${link_len} ${link_width} ${link_height}"/>
-				</geometry>
-			</visual>
-			<collision>
-				<origin xyz="0 0 0" rpy="0 0 0"/>
-				<geometry>
-					<box size="${link_len} ${link_width} ${link_height}"/>
-				</geometry>
-			</collision>
-			<xacro:inertial_matrix mass="1"/>
-		</link>
-		<gazebo reference="sixth_link">
-			<material>Gazebo/Blue</material>
-		</gazebo>
+		<link name="sixth_joint_placeholder">
+			<visual>
+				<origin xyz="0 0 0" rpy="0 0 0"/>
+				<geometry>
+					<cylinder length="0.05" radius="0.02"/>
+				</geometry>
+			</visual>
+			<collision>
+				<origin xyz="0 0 0" rpy="0 0 0"/>
+				<geometry>
+					<cylinder length="0.05" radius="0.02"/>
+				</geometry>
+			</collision>
+			<xacro:inertial_matrix mass="1"/>
+		</link>
+		<gazebo reference="sixth_joint_placeholder">
+			<material>Gazebo/Orange</material>
+		</gazebo>
+		<link name="end_effector">
+			<visual>
+				<origin xyz="0 0 0" rpy="0 0 0"/>
+				<geometry>
+					<box size="${ee_link_height} 0.010 0.015"/>
+				</geometry>
+			</visual>
+			<collision>
+				<origin xyz="0 0 0" rpy="0 0 0"/>
+				<geometry>
+					<box size="${ee_link_height} 0.010 0.015"/>
+				</geometry>
+			</collision>
+			<xacro:inertial_matrix mass="1"/>
+		</link>
+		<gazebo reference="end_effector">
+			<material>Gazebo/Black</material>
+		</gazebo>
+		<!-- JOINTS -->
 		<joint name="fixed" type="fixed">
 			<parent link="world"/>
@@ -153,37 +246,61 @@
 		</joint>
 		<joint name="second_joint" type="revolute">
-			<origin xyz="0 0 0.1" rpy="0 0 0"/>
+			<origin xyz="0 0 0.01" rpy="0 0 0"/>
 			<parent link="base_link"/>
+			<child link="second_joint_placeholder"/>
+			<axis xyz="0 0 1"/>
+			<limit effort="300" velocity="1" lower="0" upper="${M_PI}"/>
+		</joint>
+		<joint name="second_fixed" type="fixed">
+			<parent link="second_joint_placeholder"/>
 			<child link="second_link"/>
-			<axis xyz="0 0 1"/>
-			<limit effort="300" velocity="1" lower="0" upper="${M_PI}"/>
 		</joint>
 		<joint name="third_joint" type="revolute">
-			<origin xyz="0 0 0.26" rpy="${M_PI_HALVES} 0 0"/>
+			<origin xyz="0 0 0.076" rpy="0 ${-M_PI_HALVES} 0"/>
 			<parent link="second_link"/>
+			<child link="third_joint_placeholder"/>
+			<axis xyz="0 0 1"/>
+			<limit effort="300" velocity="1" lower="${-M_PI_HALVES}" upper="${M_PI_HALVES}"/>
+		</joint>
+		<joint name="third_fixed" type="fixed">
+			<origin xyz="0.034 0 0" rpy="0 0 0"/> <!-- Radius 0.03 -->
+			<parent link="third_joint_placeholder"/>
 			<child link="third_link"/>
-			<axis xyz="0 1 0"/>
-			<limit effort="300" velocity="1" lower="0" upper="${M_PI}"/>
 		</joint>
 		<joint name="fourth_joint" type="revolute">
-			<origin xyz="0 0 0.26" rpy="0 0 0"/>
+			<origin xyz="0.035 0 0" rpy="0 0 0"/>
 			<parent link="third_link"/>
+			<child link="fourth_joint_placeholder"/>
+			<axis xyz="0 0 1"/>
+			<limit effort="300" velocity="1" lower="${-M_PI_HALVES}" upper="${M_PI_HALVES}"/>
+		</joint>
+		<joint name="fourth_fixed" type="fixed">
+			<origin xyz="0.054 0 0" rpy="0 0 0"/>
+			<parent link="fourth_joint_placeholder"/>
 			<child link="fourth_link"/>
-			<axis xyz="1 0 0"/>
-			<limit effort="300" velocity="1" lower="0" upper="${M_PI}"/>
 		</joint>
 		<joint name="fifth_joint" type="revolute">
-			<origin xyz="0 0 0.26" rpy="0 0 0"/>
+			<origin xyz="0.055 0 0" rpy="0 0 0"/>
 			<parent link="fourth_link"/>
+			<child link="fifth_joint_placeholder"/>
+			<axis xyz="0 0 1"/>
+			<limit effort="300" velocity="1" lower="${-M_PI_HALVES}" upper="${M_PI_HALVES}"/>
+		</joint>
+		<joint name="fifth_fixed" type="fixed">
+			<origin xyz="0.034 0 0" rpy="0 0 0"/>
+			<parent link="fifth_joint_placeholder"/>
 			<child link="fifth_link"/>
-			<axis xyz="1 0 0"/>
-			<limit effort="300" velocity="1" lower="0" upper="${M_PI}"/>
 		</joint>
 		<joint name="sixth_joint" type="revolute">
-			<origin xyz="0 0 0.26" rpy="0 0 0"/>
+			<origin xyz="0.0275 0 0" rpy="0 0 0"/>
 			<parent link="fifth_link"/>
-			<child link="sixth_link"/>
-			<axis xyz="1 0 0"/>
-			<limit effort="300" velocity="1" lower="0" upper="${M_PI}"/>
+			<child link="sixth_joint_placeholder"/>
+			<axis xyz="0 0 1"/>
+			<limit effort="300" velocity="1" lower="${-M_PI_HALVES}" upper="${M_PI_HALVES}"/>
+		</joint>
+		<joint name="ee_joint" type="fixed">
+			<origin xyz="0.029 0 0" rpy="0 0 0"/>
+			<parent link="sixth_joint_placeholder"/>
+			<child link="end_effector"/>
 		</joint>
 		<xacro:transmission_block joint_name="second_joint"/>
@@ -194,5 +311,5 @@
 		<gazebo>
 			<plugin name="gazebo_ros_control" filename="libgazebo_ros_control.so">
-				<robotNamespace>/simple_robotic_model</robotNamespace>
+				<robotNamespace>/5dof_robot</robotNamespace>
 			</plugin>
 		</gazebo>

File: simple_robotic_model/urdf/simple_model_generated.urdf (robot description, URDF)
Before this commit: robot simple_model, 8 links, 7 joints
Links:
- removed link sixth_link
- added link fifth_joint_placeholder, mass 1; collision cylinder length=0.05 radius=0.025; visual cylinder length=0.05 radius=0.025
- added link fourth_joint_placeholder, mass 1; collision cylinder length=0.05 radius=0.025; visual cylinder length=0.05 radius=0.025
- added link second_joint_placeholder; collision cylinder length=0.021 radius=0.025; visual cylinder length=0.021 radius=0.025
- added link sixth_joint_placeholder, mass 1; collision cylinder length=0.05 radius=0.02; visual cylinder length=0.05 radius=0.02
- added link third_joint_placeholder; collision cylinder length=0.05 radius=0.025; visual cylinder length=0.05 radius=0.025
- link base_link: geometry collision box size=0.1 0.1 0.01; visual box size=0.1 0.1 0.01
- link end_effector: geometry collision box size=0.02 0.010 0.015; visual box size=0.02 0.010 0.015
- link fifth_link: geometry collision box size=0.027 0.03 0.035; visual box size=0.027 0.03 0.035
- link fourth_link: geometry collision box size=0.069 0.03 0.035; visual box size=0.069 0.03 0.035
- link second_link: geometry collision box size=0.035 0.03 0.036; visual box size=0.035 0.03 0.036
- link third_link: geometry collision box size=0.029 0.03 0.035; visual box size=0.029 0.03 0.035
Joints:
- added joint fifth_fixed: type fixed, parent fifth_joint_placeholder, child fifth_link, origin xyz=0.034 0 0 rpy=0 0 0
- added joint fourth_fixed: type fixed, parent fourth_joint_placeholder, child fourth_link, origin xyz=0.054 0 0 rpy=0 0 0
- added joint second_fixed: type fixed, parent second_joint_placeholder, child second_link
- added joint third_fixed: type fixed, parent third_joint_placeholder, child third_link, origin xyz=0.034 0 0 rpy=0 0 0
- joint ee_joint: origin xyz=0.26 0 0 rpy=0 0 0 -> xyz=0.029 0 0 rpy=0 0 0; parent sixth_link -> sixth_joint_placeholder
- joint fifth_joint: child fifth_link -> fifth_joint_placeholder; origin xyz=0.26 0 0 rpy=0 0 0 -> xyz=0.055 0 0 rpy=0 0 0
- joint fourth_joint: child fourth_link -> fourth_joint_placeholder; origin xyz=0.26 0 0 rpy=0 0 0 -> xyz=0.035 0 0 rpy=0 0 0
- joint second_joint: child second_link -> second_joint_placeholder; origin xyz=0 0 0.15 rpy=0 0 0 -> xyz=0 0 0.01 rpy=0 0 0
- joint sixth_joint: child sixth_link -> sixth_joint_placeholder; origin xyz=0.26 0 0 rpy=0 0 0 -> xyz=0.0275 0 0 rpy=0 0 0
- joint third_joint: child third_link -> third_joint_placeholder; origin xyz=0 0 0.26 rpy=0 -1.570795 0 -> xyz=0 0 0.076 rpy=0 -1.570795 0

Commit message: Update branch andré

File: simple_robotic_model/urdf/simple_model.urdf.xacro (robot description, xacro)
@@ -81,5 +81,5 @@
 		<link name="second_link">
 			<visual>
-				<origin xyz="0 0 0.039" rpy="0 0 0"/>
+				<origin xyz="0 0 0.034" rpy="0 0 0"/>
 				<geometry>
 					<box size="${link_len} ${link_width} ${second_link_height}"/>
@@ -87,5 +87,5 @@
 			</visual>
 			<collision>
-				<origin xyz="0 0 0.039" rpy="0 0 0"/>
+				<origin xyz="0 0 0.034" rpy="0 0 0"/>
 				<geometry>
 					<box size="${link_len} ${link_width} ${second_link_height}"/>

Commit message: Adjusted constraints on URDF

File: simple_robotic_model/urdf/simple_model.urdf.xacro (robot description, xacro)
@@ -261,5 +261,5 @@
 			<child link="third_joint_placeholder"/>
 			<axis xyz="0 0 1"/>
-			<limit effort="300" velocity="1" lower="${-M_PI_HALVES}" upper="${M_PI_HALVES}"/>
+			<limit effort="300" velocity="1" lower="-1.04719755" upper="1.04719755"/>
 		</joint>
 		<joint name="third_fixed" type="fixed">

File: simple_robotic_model/urdf/simple_model_generated.urdf (robot description, URDF)
Before this commit: robot simple_model, 12 links, 11 joints
Joints:
- joint third_joint: limit lower=-1.570795 upper=1.570795 effort=300 velocity=1 -> lower=-1.04719755 upper=1.04719755 effort=300 velocity=1

Commit message: Constraints

File: simple_robotic_model/urdf/simple_model.urdf.xacro (robot description, xacro)
@@ -261,5 +261,5 @@
 			<child link="third_joint_placeholder"/>
 			<axis xyz="0 0 1"/>
-			<limit effort="300" velocity="1" lower="-1.04719755" upper="1.04719755"/>
+			<limit effort="300" velocity="1" lower="${-M_PI / 4}" upper="${-M_PI / 4}"/>
 		</joint>
 		<joint name="third_fixed" type="fixed">

Commit message: ..

File: simple_robotic_model/urdf/simple_model.urdf.xacro (robot description, xacro)
@@ -261,5 +261,5 @@
 			<child link="third_joint_placeholder"/>
 			<axis xyz="0 0 1"/>
-			<limit effort="300" velocity="1" lower="${-M_PI / 4}" upper="${-M_PI / 4}"/>
+			<limit effort="300" velocity="1" lower="${-M_PI / 4}" upper="${M_PI / 4}"/>
 		</joint>
 		<joint name="third_fixed" type="fixed">

File: simple_robotic_model/urdf/simple_model_generated.urdf (robot description, URDF)
Before this commit: robot simple_model, 12 links, 11 joints
Joints:
- joint third_joint: limit lower=-0.7853975 upper=-0.7853975 effort=300 velocity=1 -> lower=-0.7853975 upper=0.7853975 effort=300 velocity=1
